File: pcb/ConversorDCDC/ConversorDCDC.sch (KiCad schematic (older format))
At the start: 26 parts, among them CN1 USBA_FEMALE, T1 MMUN2133LT1G, U1 TPS61090, X1 2.54mm, X2 3.5mm

Commit message: entrega parcial
Parts:
- removed B1: 1.8-5V, symbol Device:Battery_Cell
- removed X1: 2.54mm, Connector_JST:JST_EH_S2B-EH_1x02_P2.50mm_Horizontal, symbol Connector_Generic:Conn_01x02
- added FID1, FID2: Fiducial, Fiducial:Fiducial_0.5mm_Mask1mm, symbol Mechanical:Fiducial
- added H1, H2: MountingHole, MountingHole:MountingHole_2.2mm_M2_ISO7380_Pad_TopBottom, symbol Mechanical:MountingHole
- C1, C2, C3, C4, C6: Digikey# (none) -> 1001-2370-2-ND
- CN1: Mouser# (none) -> 640-USB1046GF0190LBA
- L1: Digikey# (none) -> 308-1566-6-ND
- LED1: Mouser# (none) -> 720-LYM676Q2S126Z
- LED2: Mouser# (none) -> 755-SML-H12V8TT86C
- R1, R10, R11, R12, R13, R2, R20, R3, R4, R5, R9: Digikey# (none) -> 2019-RK73G2ATTD33R0FDKR-ND
- T1: Digikey# (none) -> MMUN2133LT1GOSTR-ND
- U1: Digikey# (none) -> 296-15259-2-ND
- X2: Digikey# (none) -> 455-1719-ND
Connections:
- net +BATT: now also R13.2
- net ENABLE: no longer R13.2
- net GND: now also R10.2, R12.2; no longer R10.1, R12.1
- net at CN1.2 (D-), R11.2: now also R10.1; no longer R12.2
- net at CN1.3 (D+), R9.2: now also R12.1; no longer R10.2
Other:
- note added: "Conector\nBatería"
- note added: "PINES CONTROL"
- note added: "R3 = 1.9Mohm for 5.2V\nR3 = 1.87Mohm for 5.0V\nR3 = 1.1Mohm for 3.3V"
- note added: "SALIDA"
- note removed: "Both grounds must be connected on the PCB at only one point close to the GND pin"
- note removed: "R3 = 1.9Mohm for 5.2V\nR3 = 1.1Mohm for 3.3V"
- moved on the sheet: C2, C3, C6, CN1, JP1, L1, LED1, LED2, R10, R11, R12, R13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

Commit message: ruteo de pcb
Connections:
- net +BATT: no longer R13.2
- net ENABLE: now also R13.2
Changed lines of the file:
@@
 Comment1 "Trabajo práctico final"
 Comment2 "LGPL"
-Comment3 ""
+Comment3 "Circuito original: PowerBoost +1000"
 Comment4 ""
 $EndDescr
@@
 	4900 4050 5150 4050
 Connection ~ 5150 4050
-Wire Wire Line
-	4300 3250 4950 3250
 Wire Notes Line
 	3300 5200 4550 5200
@@
 $EndComp
 Wire Wire Line
-	3500 3150 4000 3150
-Wire Wire Line
 	4750 2850 4850 2850
 Connection ~ 4850 2850
@@
 Wire Wire Line
 	4000 2550 4000 2650
-Wire Wire Line
-	4000 2950 4000 3150
-Connection ~ 4000 3150
-Wire Wire Line
-	4000 3150 4400 3150
 Wire Notes Line
 	4600 2550 4750 1550
+Wire Wire Line
+	3500 3150 4400 3150
+Wire Wire Line
+	4000 2950 4000 3250
+Wire Wire Line
+	4000 3250 4950 3250
 $EndSCHEMATC
